File: canbus-mosfets-x6.kicad_sch (KiCad schematic)
At the start: 6 parts, among them J11 Conn_01x10, J2 DB9_Female_MountingHoles, J3 DB9_Male_MountingHoles, J5 Conn_01x10, J6 Conn_01x01, J7 Conn_01x10

Commit message: Adding BOM
Parts:
- J11, J5, J7: DigiKey (none) -> ED4164-64-ND
Changed lines of the file:
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@@
   (symbol (lib_id "Connector_Generic:Conn_01x10") (at 167.64 101.6 180) (unit 1)
     (in_bom yes) (on_board yes) (fields_autoplaced)
-    (property "Reference" "J11" (id 0) (at 165.1 99.0599 0)
-      (effects (font (size 1.27 1.27)) (justify left))
-    )
-    (property "Value" "Conn_01x10" (id 1) (at 165.1 101.5999 0)
+    (property "Reference" "J11" (id 0) (at 165.1 97.7899 0)
+      (effects (font (size 1.27 1.27)) (justify left))
+    )
+    (property "Value" "Conn_01x10" (id 1) (at 165.1 100.3299 0)
       (effects (font (size 1.27 1.27)) (justify left))
     )
@@
     (property "Datasheet" "~" (id 3) (at 167.64 101.6 0)
       (effects (font (size 1.27 1.27)) hide)
+    )
+    (property "DigiKey" "ED4164-64-ND" (id 4) (at 165.1 102.8699 0)
+      (effects (font (size 1.27 1.27)) (justify left))
     )
     (pin "1")
@@
       (effects (font (size 1.27 1.27)) hide)
     )
+    (property "DigiKey" "ED4164-64-ND" (id 4) (at 152.4 93.98 90))
     (pin "1")
     (pin "10")
@@
   (symbol (lib_id "Connector_Generic:Conn_01x10") (at 151.13 115.57 90) (unit 1)
     (in_bom yes) (on_board yes) (fields_autoplaced)
-    (property "Reference" "J7" (id 0) (at 152.4 109.22 90))
-    (property "Value" "Conn_01x10" (id 1) (at 152.4 111.76 90))
+    (property "Reference" "J7" (id 0) (at 152.4 106.68 90))
+    (property "Value" "Conn_01x10" (id 1) (at 152.4 109.22 90))
     (property "Footprint" "Connector_PinSocket_2.54mm:PinSocket_1x10_P2.54mm_Vertical_SMD_Pin1Left" (id 2) (at 151.13 115.57 0)
       (effects (font (size 1.27 1.27)) hide)
@@
       (effects (font (size 1.27 1.27)) hide)
     )
+    (property "DigiKey" "ED4164-64-ND" (id 4) (at 152.4 111.76 90))
     (pin "1")
     (pin "10")
