File: n-mosfet.kicad_sch (KiCad schematic)
At the start: 3 parts, among them J8 Conn_01x01, Q5 AOD4184A

Commit message: Adding BOM
Parts:
- R8: DigiKey (none) -> 311-100HRCT-ND
Changed lines of the file:
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@@
   (symbol (lib_id "Device:R_US") (at 125.73 92.71 90) (unit 1)
     (in_bom yes) (on_board yes) (fields_autoplaced)
-    (property "Reference" "R8" (id 0) (at 125.73 86.36 90))
-    (property "Value" "100" (id 1) (at 125.73 88.9 90))
+    (property "Reference" "R8" (id 0) (at 125.73 83.82 90))
+    (property "Value" "100" (id 1) (at 125.73 86.36 90))
     (property "Footprint" "Resistor_SMD:R_0603_1608Metric_Pad0.98x0.95mm_HandSolder" (id 2) (at 125.984 91.694 90)
       (effects (font (size 1.27 1.27)) hide)
@@
       (effects (font (size 1.27 1.27)) hide)
     )
+    (property "DigiKey" "311-100HRCT-ND" (id 4) (at 125.73 88.9 90))
     (pin "1")
     (pin "2")
