File: canbuz-mosfets-x6.kicad_pcb (KiCad board)
At the start: 2 copper layers, 61 x 48.3 mm, 24 parts, among them J1 Conn_01x01, J10 Conn_01x01, J11 Conn_01x10, J12 Conn_01x01, J2 DB9_Female_MountingHoles, J3 DB9_Male_MountingHoles, J4 Conn_01x01, J5 Conn_01x10, J6 Conn_01x01, J7 Conn_01x10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

Commit message: Renaming project
Other:
- board text added: "canbuz-mosfets-x6 v1.0 2022/12/01 Cedric Priscal"
- board text removed: "canbus-mosfet-x6 v1.0 2022/12/01 Cedric Priscal"
Changed lines of the file:
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@@
     (tags "9-pin D-Sub connector horizontal angled 90deg THT female pitch 2.77x2.84mm pin-PCB-offset 7.699999999999999mm mounting-holes-distance 25mm mounting-hole-offset 25mm")
     (property "DigiKey" "AE10924-ND")
-    (property "Sheetfile" "canbus-mosfets-x6.kicad_sch")
+    (property "Sheetfile" "canbuz-mosfets-x6.kicad_sch")
     (property "Sheetname" "")
     (attr through_hole)
@@
     (descr "surface-mounted straight socket strip, 1x10, 2.54mm pitch, single row, style 1 (pin 1 left) (https://cdn.harwin.com/pdfs/M20-786.pdf), script generated")
     (tags "Surface mounted socket strip SMD 1x10 2.54mm single row style1 pin1 left")
-    (property "Sheetfile" "canbus-mosfets-x6.kicad_sch")
+    (property "Sheetfile" "canbuz-mosfets-x6.kicad_sch")
     (property "Sheetname" "")
     (attr smd)
@@
     (tags "9-pin D-Sub connector horizontal angled 90deg THT male pitch 2.77x2.84mm pin-PCB-offset 7.699999999999999mm mounting-holes-distance 25mm mounting-hole-offset 25mm")
     (property "DigiKey" "AE10970-ND")
-    (property "Sheetfile" "canbus-mosfets-x6.kicad_sch")
+    (property "Sheetfile" "canbuz-mosfets-x6.kicad_sch")
     (property "Sheetname" "")
     (attr through_hole)
@@
     (descr "surface-mounted straight socket strip, 1x10, 2.54mm pitch, single row, style 1 (pin 1 left) (https://cdn.harwin.com/pdfs/M20-786.pdf), script generated")
     (tags "Surface mounted socket strip SMD 1x10 2.54mm single row style1 pin1 left")
-    (property "Sheetfile" "canbus-mosfets-x6.kicad_sch")
+    (property "Sheetfile" "canbuz-mosfets-x6.kicad_sch")
     (property "Sheetname" "")
     (attr smd)
@@
     (descr "surface-mounted straight socket strip, 1x10, 2.54mm pitch, single row, style 1 (pin 1 left) (https://cdn.harwin.com/pdfs/M20-786.pdf), script generated")
     (tags "Surface mounted socket strip SMD 1x10 2.54mm single row style1 pin1 left")
-    (property "Sheetfile" "canbus-mosfets-x6.kicad_sch")
+    (property "Sheetfile" "canbuz-mosfets-x6.kicad_sch")
     (property "Sheetname" "")
     (attr smd)
@@
     (descr "Soldered wire connection, for a single 1 mm² wire, reinforced insulation, conductor diameter 1.4mm, outer diameter 3.9mm, size source Multi-Contact FLEXI-xV 1.0 (https://ec.staubli.com/AcroFiles/Catalogues/TM_Cab-Main-11014119_(en)_hi.pdf), bend radius 3 times outer diameter, generated with kicad-footprint-generator")
     (tags "connector wire 1sqmm")
-    (property "Sheetfile" "canbus-mosfets-x6.kicad_sch")
+    (property "Sheetfile" "canbuz-mosfets-x6.kicad_sch")
     (property "Sheetname" "")
     (attr exclude_from_pos_files)
@@
     (effects (font (size 1 1) (thickness 0.15)))
   )
-  (gr_text "canbus-mosfet-x6\nv1.0 2022/12/01\nCedric Priscal" (at 180.792 151.788) (layer "F.SilkS")
+  (gr_text "canbuz-mosfets-x6\nv1.0 2022/12/01\nCedric Priscal" (at 180.792 151.788) (layer "F.SilkS")
     (effects (font (size 1 1) (thickness 0.15)) (justify right))
   )
